Commit message: split the single and multi

File: jackal_description/urdf/accessories/ns_sick_lms1xx_upright_mount.urdf.xacro (robot description, xacro)
@@ -27,6 +27,6 @@
 <robot xmlns:xacro="http://www.ros.org/wiki/xacro">
   <xacro:include filename="$(find lms1xx)/urdf/sick_lms1xx.urdf.xacro" />
-  <xacro:macro name="sick_lms1xx_upright_mount" params="prefix topic parent_link *origin">
-    <xacro:sick_lms1xx frame="${prefix}_laser" topic="${topic}" />
+  <xacro:macro name="ns_sick_lms1xx_upright_mount" params="prefix topic parent_link *origin">
+    <xacro:sick_lms1xx frame="${prefix}_laser" topic="${topic}" robot_namespace="$(arg namespace)" />
     <joint name="${prefix}_laser_mount_joint" type="fixed">
       <xacro:insert_block name="origin" />
